File: pls work/pls work.kicad_pcb (KiCad board)
At the start: 2 copper layers, 72 parts, among them J1 ST7735R, J2 SD Card, SW1 RotaryEncoder_Switch_MP, SW10 SW_Push_45deg, SW11 SW_Push_45deg, SW12 SW_Push_45deg, SW13 SW_Push_45deg, SW14 SW_Push_45deg, SW15 SW_Push_45deg, SW16 SW_Push_45deg, SW17 SW_Push_45deg, SW18 SW_Push_45deg, SW19 SW_Push_45deg, SW2 RotaryEncoder_Switch_MP, SW20 SW_Push_45deg, SW21 SW_Push_45deg, SW22 SW_Push_45deg, SW23 SW_Push_45deg, SW24 SW_Push_45deg, SW25 SW_Push_45deg, SW26 SW_Push_45deg, SW27 SW_Push_45deg, SW28 SW_Push_45deg, SW29 SW_Push_45deg, SW3 SW_Push_45deg, SW30 SW_Push_45deg, SW31 SW_Push_45deg, SW32 SW_Push_45deg, SW33 SW_Push_45deg, SW34 SW_Push_45deg, SW35 SW_Push_45deg, SW36 SW_Push_45deg, SW4 SW_Push_45deg, SW5 SW_Push_45deg, SW6 SW_Push_45deg, SW7 SW_Push_45deg, SW8 SW_Push_45deg, SW9 SW_Push_45deg

Commit message: WIRING
soooo much wiring
Parts:
- J2: footprint Connector:FanPinHeader_1x04_P2.54mm_Vertical -> Connector_PinHeader_1.00mm:PinHeader_1x04_P1.00mm_Vertical
- moved SW1 96.2 mm to (250.2, 70.0), turned to 90 degrees
- moved SW28 96.1 mm to (274.1, 87.4)
- moved SW2 88.7 mm to (265.5, 70.0), turned to 90 degrees
- moved A1 61.7 mm to (214.7, 56.2)
- moved J2 57.2 mm to (200.5, 61.5)
- moved J1 46.3 mm to (206.5, 58.0)
Routing:
- net /ROW3: track 0.00 -> 741.5 mm
- net /ROW0: track 0.00 -> 304.5 mm
- net /ROW1: track 0.00 -> 243.7 mm
- net /COL3: track 0.00 -> 226.7 mm
- net GND: track 0.00 -> 171.1 mm
- net /COL1: track 0.00 -> 148.0 mm
- net /2B: track 0.00 -> 134.8 mm
- net /ROW2: track 0.00 -> 93.7 mm
- net /2A: track 0.00 -> 92.1 mm
- net /1B: track 0.00 -> 89.1 mm
- net /COL2: track 0.00 -> 85.8 mm
- net /COL0: track 0.00 -> 82.2 mm
- net /ROW4: track 0.00 -> 76.9 mm
- net /1A: track 0.00 -> 73.8 mm
- net /A0: track 0.00 -> 64.7 mm
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Other:
- board outline added: 310.4 x 115.6 mm

Commit message: wiring is NOT working
restarting now trying to come up with a better plan
Parts:
- moved D11 14.0 mm to (225.2, 139.0)
- moved D18 14.0 mm to (240.0, 138.5)
- moved D25 14.0 mm to (254.9, 139.0)
- moved D31 14.0 mm to (270.5, 139.0)
- moved D32 14.0 mm to (190.7, 139.0)
- moved D4 14.0 mm to (209.4, 139.0)
- moved SW13 14.0 mm to (231.2, 141.9)
- moved SW27 14.0 mm to (261.4, 141.9)
- moved SW34 14.0 mm to (276.5, 141.9)
- moved SW35 14.0 mm to (196.5, 141.9)
- moved SW6 14.0 mm to (216.1, 141.9)
- moved SW20 14.0 mm to (246.3, 141.9)
Routing:
- net /ROW3: track 741.5 -> 0.00 mm
- net /ROW0: track 304.5 -> 0.00 mm
- net /ROW1: track 243.7 -> 0.00 mm
- net /COL3: track 226.7 -> 0.00 mm
- net GND: track 171.1 -> 0.00 mm
- net /COL1: track 148.0 -> 0.00 mm
- net /2B: track 134.8 -> 0.00 mm
- net /ROW2: track 93.7 -> 0.00 mm
- net /2A: track 92.1 -> 0.00 mm
- net /1B: track 89.1 -> 0.00 mm
- net /COL2: track 85.8 -> 0.00 mm
- net /COL0: track 82.2 -> 0.00 mm
- net /ROW4: track 76.9 -> 0.00 mm
- net /1A: track 73.8 -> 0.00 mm
- net /A0: track 64.7 -> 0.00 mm
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Other:
- board size 310.4 x 115.6 mm -> 301.1 x 115.6 mm

Commit message: still wiring...
these wires r killing meee
Parts:
- moved D31 238.5 mm to (36.0, 95.5)
- moved SW34 238.5 mm to (42.0, 98.4)
- moved D28 216.8 mm to (55.5, 72.0)
- moved SW31 216.8 mm to (61.1, 75.4)
- moved SW28 196.3 mm to (80.5, 55.4)
- moved D1 190.7 mm to (16.9, 119.0)
- moved SW3 190.7 mm to (23.0, 122.4)
- moved D7 189.6 mm to (35.5, 144.0)
- moved SW10 189.6 mm to (41.5, 146.9)
- moved D20 171.2 mm to (264.7, 143.5)
- moved SW22 171.2 mm to (271.0, 146.9)
- moved D17 146.2 mm to (207.9, 143.5)
- moved SW19 146.2 mm to (214.0, 146.9)
- moved D32 142.3 mm to (55.2, 95.5)
- moved SW35 142.3 mm to (61.0, 98.4)
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Routing:
- net /COL3: track 0.00 -> 413.3 mm
- net /COL2: track 0.00 -> 334.9 mm
- net /ROW2: track 0.00 -> 327.5 mm
- net /ROW1: track 0.00 -> 303.5 mm
- net /COL1: track 0.00 -> 275.2 mm
- net /ROW3: track 0.00 -> 274.4 mm
- net /ROW0: track 0.00 -> 262.9 mm
- net /COL0: track 0.00 -> 246.9 mm
- net /COL5: track 0.00 -> 232.8 mm
- net /COL4: track 0.00 -> 218.2 mm
- net /COL6: track 0.00 -> 196.4 mm
- net GND: track 0.00 -> 182.9 mm
- net /ROW4: track 0.00 -> 81.8 mm
- net /1A: track 0.00 -> 81.2 mm
- net Net-(A1-RUN): track 0.00 -> 52.1 mm
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
Commit message: done the wiring
but got like 140 warnings...
Routing:
- net GND: track 182.9 -> 238.7 mm
- net /MOSI: track 10.7 -> 44.9 mm
- net /COL2: track 334.9 -> 362.5 mm
- net /COL3: track 413.3 -> 436.2 mm
- net /1B: track 30.2 -> 48.2 mm
- net +3V3: track 0.00 -> 8.43 mm
- net /COL5: track 232.8 -> 238.1 mm
- net /CS_LCD: track 12.2 -> 7.47 mm
- net /SCK: track 39.0 -> 42.6 mm
- net /1A: track 81.2 -> 79.1 mm
- net /A0: track 9.95 -> 11.3 mm
Other:
- board text added: "Steinway & Sons"

Commit message: ok now my error fixing work is showing up
Parts:
- moved D23 2.04 mm to (196.9, 117.5)
- moved D25 2.04 mm to (234.9, 117.5)
- moved D22 2.01 mm to (159.4, 118.0)
- moved D21 2.00 mm to (141.0, 118.0)
- moved D24 1.51 mm to (215.9, 117.5)
- moved D33 1.12 mm to (74.9, 94.5)
- moved D9 1.00 mm to (106.4, 119.0)
- moved D4 0.74 mm to (86.7, 119.5)
- moved D27 0.71 mm to (36.4, 72.0)
- moved D12 0.55 mm to (111.9, 143.5)
- moved D29 0.50 mm to (74.5, 72.0)
- moved D32 0.50 mm to (55.2, 95.0)
- moved D7 0.50 mm to (35.5, 143.5)
Routing:
- net /COL5: track 238.1 -> 270.9 mm
- net /1A: track 79.1 -> 64.0 mm
- net /COL1: track 275.2 -> 271.9 mm
- net Net-(D25-A): track 3.39 -> 5.56 mm
- net Net-(D23-A): track 3.39 -> 5.56 mm
- net Net-(D21-A): track 3.69 -> 5.69 mm
- net Net-(D24-A): track 4.14 -> 5.73 mm
- net /COL3: track 436.2 -> 437.4 mm
- net Net-(D33-A): track 10.7 -> 11.9 mm
- net Net-(D9-A): track 9.63 -> 10.3 mm
- net /COL6: track 196.4 -> 197.1 mm
Other:
- board text removed: "Steinway & Sons"

Commit message: fixed most of my issues
just a few spacing problems that I will have to figure out later
Parts:
- moved D11 0.92 mm to (92.7, 143.5)
- moved D31 0.53 mm to (36.2, 95.0)
- moved D14 0.50 mm to (150.1, 143.5)
- moved D5 0.50 mm to (-3.26, 143.5)
Connections:
- D21 pad 1: unconnected-(D21-K-Pad1) -> /COL1
- D22 pad 1: unconnected-(D22-K-Pad1) -> /COL2
- D23 pad 1: unconnected-(D23-K-Pad1) -> /COL4
- D24 pad 1: unconnected-(D24-K-Pad1) -> /COL5
- D25 pad 1: unconnected-(D25-K-Pad1) -> /COL6
Routing:
- net /COL4: track 218.2 -> 256.4 mm, vias 0 -> 1
- net /COL6: track 197.1 -> 227.8 mm
- net /COL2: track 362.7 -> 391.7 mm
- net /COL1: track 271.9 -> 299.5 mm
- net /COL0: track 246.9 -> 266.9 mm
- net /ROW3: track 274.4 -> 289.5 mm
- net /COL3: track 437.4 -> 446.4 mm
- net Net-(D22-A): track 3.44 -> 5.52 mm
- net /ROW0: track 262.9 -> 264.6 mm
- net GND: track 238.7 -> 239.9 mm
- net /COL5: track 270.9 -> 270.1 mm
- net Net-(D11-A): track 10.2 -> 9.67 mm
