File: pls work/pls work.kicad_sch (KiCad schematic)
At the start: 55 parts, among them J1 ST7735R, SW1 RotaryEncoder_Switch_MP, SW10 SW_Push_45deg, SW11 SW_Push_45deg, SW12 SW_Push_45deg, SW13 SW_Push_45deg, SW14 SW_Push_45deg, SW15 SW_Push_45deg, SW16 SW_Push_45deg, SW17 SW_Push_45deg, SW18 SW_Push_45deg, SW19 SW_Push_45deg, SW2 RotaryEncoder_Switch_MP, SW20 SW_Push_45deg, SW21 SW_Push_45deg, SW22 SW_Push_45deg, SW23 SW_Push_45deg, SW24 SW_Push_45deg, SW25 SW_Push_45deg, SW26 SW_Push_45deg, SW27 SW_Push_45deg, SW28 SW_Push_45deg, SW3 SW_Push_45deg, SW4 SW_Push_45deg, SW5 SW_Push_45deg, SW6 SW_Push_45deg, SW7 SW_Push_45deg, SW8 SW_Push_45deg, SW9 SW_Push_45deg

Commit message: still working on schematic stuff
still got a bunch to do... idk im doing it right
Parts:
- added J2: SD Card, symbol Connector:Conn_01x04_Pin
Connections:
- net SCK: now also J2.1 (Pin_1)
- new net DATA: J2.3 (Pin_3)
- new net LRCK: J2.2 (Pin_2)
Other:
- moved on the sheet: D13, D14, D15, D16, D17, D18, D19, D20, D21, D22, D23, D24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

Commit message: finished schematic (hopefully), did footprints, now doing pcb
struggling not too bad rn tho
Parts:
- added D26, D27, D28, D29, D30, D31, D32, D33: 1N4148, Diode_THT:D_DO-35_SOD27_P7.62mm_Horizontal, symbol Diode:1N4148
- added SW29, SW30, SW31, SW32, SW33, SW34, SW35, SW36: SW_Push_45deg, Button_Switch_Keyboard:SW_Cherry_MX_1.00u_PCB, symbol Switch:SW_Push_45deg
- A1: footprint Module:RaspberryPi_Pico_Common_Unspecified -> Module:RaspberryPi_Pico_Common_THT
- J1: footprint (none) -> Connector_PinHeader_1.00mm:PinHeader_1x08_P1.00mm_Vertical
- J2: footprint (none) -> Connector:FanPinHeader_1x04_P2.54mm_Vertical
- SW1, SW2: footprint (none) -> Rotary_Encoder:RotaryEncoder_Alps_EC11E-Switch_Vertical_H20mm_MountingHoles
- SW10, SW11, SW12, SW13, SW14, SW15, SW16, SW17, SW18, SW19, SW20, SW21, SW22, SW23, SW24, SW25, SW26, SW27, SW28, SW3, SW4, SW5, SW6, SW7, SW8, SW9: footprint (none) -> Button_Switch_Keyboard:SW_Cherry_MX_1.00u_PCB
Connections:
- net DATA is gone; now on net MISO: J2.3 (Pin_3)
- net LRCK is gone; now on net MOSI: J2.2 (Pin_2)
- net ROW5 is gone; now on net COL3: A1.7 (GPIO5)
- net COL0: now also D26.1 (K), D30.1 (K)
- net COL1: now also D27.1 (K), D31.1 (K)
- net COL2: now also D28.1 (K), D32.1 (K)
- net COL3: now also D29.1 (K), D33.1 (K), SW33.1, SW34.1, SW35.1, SW36.1
- net GND: now also A1.33 (AGND)
- net ROW4: now also SW29.1, SW30.1, SW31.1, SW32.1
- net CS: now reaches J2.4 (Pin_4)
- new net: D28.2 (A), SW31.2
- new net: D33.2 (A), SW36.2
- new net: D26.2 (A), SW29.2
- new net: D30.2 (A), SW33.2
- new net: D32.2 (A), SW35.2
- new net: D31.2 (A), SW34.2
- new net: D29.2 (A), SW32.2
- new net: D27.2 (A), SW30.2
- no-connect marks 2 -> 1
Other:
- moved on the sheet: A1, SW28

Commit message: WIRING
soooo much wiring
Parts:
- J2: footprint Connector:FanPinHeader_1x04_P2.54mm_Vertical -> Connector_PinHeader_1.00mm:PinHeader_1x04_P1.00mm_Vertical
Changed lines of the file:
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@@
 			)
 		)
-		(property "Footprint" "Connector:FanPinHeader_1x04_P2.54mm_Vertical"
+		(property "Footprint" "Connector_PinHeader_1.00mm:PinHeader_1x04_P1.00mm_Vertical"
 			(at 138.43 25.4 0)
 			(hide yes)

Commit message: fixed most of my issues
just a few spacing problems that I will have to figure out later
Connections:
- net COL1: now also D21.1 (K)
- net COL2: now also D22.1 (K)
- net COL4: now also D23.1 (K)
- net COL5: now also D24.1 (K)
- net COL6: now also D25.1 (K)
Changed lines of the file:
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@@
+	)
+	(junction
+		(at 100.33 113.03)
+		(diameter 0)
+		(color 0 0 0 0)
 	)
 	(junction
@@
 	)
 	(junction
+		(at 68.58 113.03)
+		(diameter 0)
+		(color 0 0 0 0)
+	)
+	(junction
 		(at 62.23 83.82)
 		(diameter 0)
@@
 	)
 	(junction
+		(at 54.61 113.03)
+		(diameter 0)
+		(color 0 0 0 0)
+	)
+	(junction
 		(at 54.61 44.45)
 		(diameter 0)
@@
 	)
 	(junction
+		(at 129.54 113.03)
+		(diameter 0)
+		(color 0 0 0 0)
+	)
+	(junction
 		(at 55.88 118.11)
 		(diameter 0)
@@
 	(junction
 		(at 52.07 132.08)
+		(diameter 0)
+		(color 0 0 0 0)
+	)
+	(junction
+		(at 115.57 113.03)
 		(diameter 0)
 		(color 0 0 0 0)
@@
 	(wire
 		(pts
+			(xy 106.68 127) (xy 113.03 127)
+		)
+		(stroke
+			(width 0)
+			(type default)
+		)
+	)
+	(wire
+		(pts
 			(xy 40.64 149.86) (xy 40.64 163.83)
 		)
@@
 	(wire
 		(pts
+			(xy 100.33 105.41) (xy 100.33 113.03)
+		)
+		(stroke
+			(width 0)
+			(type default)
+		)
+	)
+	(wire
+		(pts
 			(xy 27.94 158.75) (xy 45.72 158.75)
 		)
@@
 	(wire
 		(pts
+			(xy 54.61 113.03) (xy 54.61 127)
+		)
+		(stroke
+			(width 0)
+			(type default)
+		)
+	)
+	(wire
+		(pts
 			(xy 77.47 73.66) (xy 77.47 83.82)
 		)
@@
 	(wire
 		(pts
+			(xy 121.92 127) (xy 129.54 127)
+		)
+		(stroke
+			(width 0)
+			(type default)
+		)
+	)
+	(wire
+		(pts
 			(xy 57.15 73.66) (xy 62.23 73.66)
 		)
@@
 	(wire
 		(pts
+			(xy 68.58 119.38) (xy 68.58 113.03)
+		)
+		(stroke
+			(width 0)
+			(type default)
+		)
+	)
+	(wire
+		(pts
 			(xy 74.93 149.86) (xy 74.93 163.83)
 		)
@@
 	(wire
 		(pts
+			(xy 48.26 127) (xy 54.61 127)
+		)
+		(stroke
+			(width 0)
+			(type default)
+		)
+	)
+	(wire
+		(pts
 			(xy 58.42 149.86) (xy 58.42 163.83)
 		)
@@
 	(wire
 		(pts
+			(xy 64.77 119.38) (xy 68.58 119.38)
+		)
+		(stroke
+			(width 0)
+			(type default)
+		)
+	)
+	(wire
+		(pts
 			(xy 62.23 158.75) (xy 78.74 158.75)
 		)
@@
 	(wire
 		(pts
+			(xy 91.44 119.38) (xy 100.33 119.38)
+		)
+		(stroke
+			(width 0)
+			(type default)
+		)
+	)
+	(wire
+		(pts
 			(xy 55.88 118.11) (xy 72.39 118.11)
 		)
@@
 	(wire
 		(pts
+			(xy 113.03 119.38) (xy 115.57 119.38)
+		)
+		(stroke
+			(width 0)
+			(type default)
+		)
+	)
+	(wire
+		(pts
+			(xy 113.03 127) (xy 113.03 119.38)
+		)
+		(stroke
+			(width 0)
+			(type default)
+		)
+	)
+	(wire
+		(pts
 			(xy 93.98 132.08) (xy 109.22 132.08)
 		)
@@
 	(wire
 		(pts
+			(xy 115.57 113.03) (xy 115.57 119.38)
+		)
+		(stroke
+			(width 0)
+			(type default)
+		)
+	)
+	(wire
+		(pts
 			(xy 115.57 105.41) (xy 115.57 113.03)
 		)
@@
 	(wire
 		(pts
+			(xy 91.44 127) (xy 91.44 119.38)
+		)
+		(stroke
+			(width 0)
+			(type default)
+		)
+	)
+	(wire
+		(pts
 			(xy 74.93 163.83) (xy 74.93 167.64)
 		)
@@
 	(wire
 		(pts
+			(xy 64.77 127) (xy 64.77 119.38)
+		)
+		(stroke
+			(width 0)
+			(type default)
+		)
+	)
+	(wire
+		(pts
+			(xy 129.54 127) (xy 129.54 113.03)
+		)
+		(stroke
+			(width 0)
+			(type default)
+		)
+	)
+	(wire
+		(pts
 			(xy 62.23 83.82) (xy 62.23 88.9)
 		)
@@
 	(wire
 		(pts
+			(xy 100.33 113.03) (xy 100.33 119.38)
+		)
+		(stroke
+			(width 0)
+			(type default)
+		)
+	)
+	(wire
+		(pts
 			(xy 52.07 132.08) (xy 78.74 132.08)
 		)
@@
 		)
 		(stroke
-			(width 0)
-			(type default)
-		)
-	)
-	(wire
-		(pts
-			(xy 100.33 105.41) (xy 100.33 113.03)
-		)
-		(stroke
